Commit message: update URDF

File: urdf/apex_hand_right.urdf (robot description, URDF)
Before this commit: robot apex_hand_right, 47 links, 46 joints
Links:
- removed link Palm_link_right
- removed link f0_link0
- removed link f0_link1
- removed link f0_link2
- removed link f0_link2sensor
- removed link f0_link3
- removed link f0_link3sensor
- removed link f0_link4
- removed link f0_link4sensor
- removed link f0_pad
- removed link f0_tip
- removed link f1_link0
- removed link f1_link1
- removed link f1_link1sensor
- removed link f1_link2
- removed link f1_link2sensor
- removed link f1_link3
- removed link f1_link3sensor
- removed link f1_pad
- removed link f1_tip
- removed link f2_link0
- removed link f2_link1
- removed link f2_link1sensor
- removed link f2_link2
- removed link f2_link2sensor
- removed link f2_link3
- removed link f2_link3sensor
- removed link f2_pad
- removed link f2_tip
- removed link f3_link0
- removed link f3_link1
- removed link f3_link1sensor
- removed link f3_link2
- removed link f3_link2sensor
- removed link f3_link3
- removed link f3_link3sensor
- removed link f3_pad
- removed link f3_tip
- removed link f4_link0
- removed link f4_link1
- removed link f4_link1sensor
- removed link f4_link2
- removed link f4_link2sensor
- removed link f4_link3
- removed link f4_link3sensor
- removed link f4_pad
- removed link f4_tip
- added link right_index_link0, mass 0.018794; collision mesh filename=./meshes/right_index_link0.STL; visual mesh filename=./meshes/right_index_link0.STL
- added link right_index_link1, mass 0.029095; collision mesh filename=./meshes/right_index_link1.STL; visual mesh filename=./meshes/right_index_link1.STL
- added link right_index_link2, mass 0.011142; collision mesh filename=./meshes/right_index_link2.STL; visual mesh filename=./meshes/right_index_link2.STL
- added link right_index_link3, mass 0.005232; collision mesh filename=./meshes/right_index_link3.STL; visual mesh filename=./meshes/right_index_link3.STL
- added link right_index_pad, mass 7.85398163397449E-07; collision mesh filename=./meshes/right_index_pad.STL; visual mesh filename=./meshes/right_index_pad.STL
- added link right_index_tactile0, mass 0.008926; collision mesh filename=./meshes/right_index_tactile0.STL; visual mesh filename=./meshes/right_index_tactile0.STL
- added link right_index_tactile1, mass 0.003635; collision mesh filename=./meshes/right_index_tactile1.STL; visual mesh filename=./meshes/right_index_tactile1.STL
- added link right_index_tactile2, mass 0.009866; collision mesh filename=./meshes/right_index_tactile2.STL; visual mesh filename=./meshes/right_index_tactile2.STL
- added link right_index_tip, mass 9.81747704246811E-08; collision mesh filename=./meshes/right_index_tip.STL; visual mesh filename=./meshes/right_index_tip.STL
- added link right_middle_link0, mass 0.018794; collision mesh filename=./meshes/right_middle_link0.STL; visual mesh filename=./meshes/right_middle_link0.STL
- added link right_middle_link1, mass 0.029095; collision mesh filename=./meshes/right_middle_link1.STL; visual mesh filename=./meshes/right_middle_link1.STL
- added link right_middle_link2, mass 0.011142; collision mesh filename=./meshes/right_middle_link2.STL; visual mesh filename=./meshes/right_middle_link2.STL
- added link right_middle_link3, mass 0.005232; collision mesh filename=./meshes/right_middle_link3.STL; visual mesh filename=./meshes/right_middle_link3.STL
- added link right_middle_pad, mass 7.85398163397448E-07; collision mesh filename=./meshes/right_middle_pad.STL; visual mesh filename=./meshes/right_middle_pad.STL
- added link right_middle_tactile0, mass 0.008926; collision mesh filename=./meshes/right_middle_tactile0.STL; visual mesh filename=./meshes/right_middle_tactile0.STL
- added link right_middle_tactile1, mass 0.003635; collision mesh filename=./meshes/right_middle_tactile1.STL; visual mesh filename=./meshes/right_middle_tactile1.STL
- added link right_middle_tactile2, mass 0.009866; collision mesh filename=./meshes/right_middle_tactile2.STL; visual mesh filename=./meshes/right_middle_tactile2.STL
- added link right_middle_tip, mass 9.81747704246811E-08; collision mesh filename=./meshes/right_middle_tip.STL; visual mesh filename=./meshes/right_middle_tip.STL
- added link right_palm_base, mass 0.1; collision mesh filename=./meshes/right_palm_base.STL; visual mesh filename=./meshes/right_palm_base.STL
- added link right_palm_link, mass 0.2; collision mesh filename=./meshes/right_palm_link.STL; visual mesh filename=./meshes/right_palm_link.STL
- added link right_palm_tactile, mass 0; collision mesh filename=./meshes/right_palm_tactile.STL; visual mesh filename=./meshes/right_palm_tactile.STL
- added link right_pinky_link0, mass 0.018794; collision mesh filename=./meshes/right_pinky_link0.STL; visual mesh filename=./meshes/right_pinky_link0.STL
- added link right_pinky_link1, mass 0.029095; collision mesh filename=./meshes/right_pinky_link1.STL; visual mesh filename=./meshes/right_pinky_link1.STL
- added link right_pinky_link2, mass 0.011142; collision mesh filename=./meshes/right_pinky_link2.STL; visual mesh filename=./meshes/right_pinky_link2.STL
- added link right_pinky_link3, mass 0.005232; collision mesh filename=./meshes/right_pinky_link3.STL; visual mesh filename=./meshes/right_pinky_link3.STL
- added link right_pinky_pad, mass 7.85398163397449E-07; collision mesh filename=./meshes/right_pinky_pad.STL; visual mesh filename=./meshes/right_pinky_pad.STL
- added link right_pinky_tactile0, mass 0.008926; collision mesh filename=./meshes/right_pinky_tactile0.STL; visual mesh filename=./meshes/right_pinky_tactile0.STL
- added link right_pinky_tactile1, mass 0.003635; collision mesh filename=./meshes/right_pinky_tactile1.STL; visual mesh filename=./meshes/right_pinky_tactile1.STL
- added link right_pinky_tactile2, mass 0.009866; collision mesh filename=./meshes/right_pinky_tactile2.STL; visual mesh filename=./meshes/right_pinky_tactile2.STL
- added link right_pinky_tip, mass 9.81747704246811E-08; collision mesh filename=./meshes/right_pinky_tip.STL; visual mesh filename=./meshes/right_pinky_tip.STL
- added link right_ring_link0, mass 0.018794; collision mesh filename=./meshes/right_ring_link0.STL; visual mesh filename=./meshes/right_ring_link0.STL
- added link right_ring_link1, mass 0.029095; collision mesh filename=./meshes/right_ring_link1.STL; visual mesh filename=./meshes/right_ring_link1.STL
- added link right_ring_link2, mass 0.011142; collision mesh filename=./meshes/right_ring_link2.STL; visual mesh filename=./meshes/right_ring_link2.STL
- added link right_ring_link3, mass 0.005232; collision mesh filename=./meshes/right_ring_link3.STL; visual mesh filename=./meshes/right_ring_link3.STL
- added link right_ring_pad, mass 7.85398163397448E-07; collision mesh filename=./meshes/right_ring_pad.STL; visual mesh filename=./meshes/right_ring_pad.STL
- added link right_ring_tactile0, mass 0.008926; collision mesh filename=./meshes/right_ring_tactile0.STL; visual mesh filename=./meshes/right_ring_tactile0.STL
- added link right_ring_tactile1, mass 0.003635; collision mesh filename=./meshes/right_ring_tactile1.STL; visual mesh filename=./meshes/right_ring_tactile1.STL
- added link right_ring_tactile2, mass 0.009866; collision mesh filename=./meshes/right_ring_tactile2.STL; visual mesh filename=./meshes/right_ring_tactile2.STL
- added link right_ring_tip, mass 9.81747704246808E-08; collision mesh filename=./meshes/right_ring_tip.STL; visual mesh filename=./meshes/right_ring_tip.STL
- added link right_thumb_link0, mass 0.01096758; collision mesh filename=./meshes/right_thumb_link0.STL; visual mesh filename=./meshes/right_thumb_link0.STL
- added link right_thumb_link1, mass 0.01551203; collision mesh filename=./meshes/right_thumb_link1.STL; visual mesh filename=./meshes/right_thumb_link1.STL
- added link right_thumb_link2, mass 0.0324231; collision mesh filename=./meshes/right_thumb_link2.STL; visual mesh filename=./meshes/right_thumb_link2.STL
- added link right_thumb_link3, mass 0.018383721; collision mesh filename=./meshes/right_thumb_link3.STL; visual mesh filename=./meshes/right_thumb_link3.STL
- added link right_thumb_link4, mass 0.007655847; collision mesh filename=./meshes/right_thumb_link4.STL; visual mesh filename=./meshes/right_thumb_link4.STL
- added link right_thumb_pad, mass 3.927E-07; collision mesh filename=./meshes/right_thumb_pad.STL; visual mesh filename=./meshes/right_thumb_pad.STL
- added link right_thumb_tactile0, mass 0.035995576; collision mesh filename=./meshes/right_thumb_tactile0.STL; visual mesh filename=./meshes/right_thumb_tactile0.STL
- added link right_thumb_tactile1, mass 0.0093845355; collision mesh filename=./meshes/right_thumb_tactile1.STL; visual mesh filename=./meshes/right_thumb_tactile1.STL
- added link right_thumb_tactile2, mass 0.0098665; collision mesh filename=./meshes/right_thumb_tactile2.STL; visual mesh filename=./meshes/right_thumb_tactile2.STL
- added link right_thumb_tip, mass 4.90873852123406E-08; collision mesh filename=./meshes/right_thumb_tip.STL; visual mesh filename=./meshes/right_thumb_tip.STL
Joints:
- removed joint f0_joint0
- removed joint f0_joint1
- removed joint f0_joint2
- removed joint f0_joint2sensor
- removed joint f0_joint3
- removed joint f0_joint3sensor
- removed joint f0_joint4
- removed joint f0_joint4sensor
- removed joint f0_pad
- removed joint f0_tip
- removed joint f1_joint0
- removed joint f1_joint1
- removed joint f1_joint1sensor
- removed joint f1_joint2
- removed joint f1_joint2sensor
- removed joint f1_joint3
- removed joint f1_joint3sensor
- removed joint f1_pad
- removed joint f1_tip
- removed joint f2_joint0
- removed joint f2_joint1
- removed joint f2_joint1sensor
- removed joint f2_joint2
- removed joint f2_joint2sensor
- removed joint f2_joint3
- removed joint f2_joint3sensor
- removed joint f2_pad
- removed joint f2_tip
- removed joint f3_joint0
- removed joint f3_joint1
- removed joint f3_joint2
- removed joint f3_joint2sensor
- removed joint f3_joint3
- removed joint f3_joint3sensor
- removed joint f3_link1sensor
- removed joint f3_pad
- removed joint f3_tip
- removed joint f4_joint0
- removed joint f4_joint1
- removed joint f4_joint1sensor
- removed joint f4_joint2
- removed joint f4_joint3
- removed joint f4_joint3sensor
- removed joint f4_link2sensor
- removed joint f4_pad
- removed joint f4_tip
- added joint right_index_j0: type revolute, parent right_palm_base, child right_index_link0, origin xyz=0.0071 0.034496 0.1188 rpy=0 -1.5708 0, axis 0 0 1, limit lower=-0.4363 upper=0.4363 effort=0 velocity=0
- added joint right_index_j1: type revolute, parent right_index_link0, child right_index_link1, origin xyz=0.016 0 0 rpy=-1.5708 0 0, axis 0 0 1, limit lower=-0.349 upper=1.5707 effort=0 velocity=0
- added joint right_index_j2: type revolute, parent right_index_link1, child right_index_link2, origin xyz=0.045 0 0 rpy=0 0 0, axis 0 0 1, limit lower=-0.0872 upper=1.7453 effort=0 velocity=0
- added joint right_index_j3: type revolute, parent right_index_link2, child right_index_link3, origin xyz=0.025 0 0 rpy=0 0 0, axis 0 0 1, limit lower=-0.0872 upper=1.7453 effort=0 velocity=0, mimic joint=right_index_j2 multiplier=1.0 offset=0
- added joint right_index_pad_fix: type fixed, parent right_index_tactile2, child right_index_pad, origin xyz=0.017096 0.0071955 0 rpy=0 0 0, axis 0 0 0
- added joint right_index_tactile0_fix: type fixed, parent right_index_link1, child right_index_tactile0, origin xyz=0 0 0 rpy=0 0 0, axis 0 0 0
- added joint right_index_tactile1_fix: type fixed, parent right_index_link2, child right_index_tactile1, origin xyz=0 0 0 rpy=0 0 0, axis 0 0 0
- added joint right_index_tactile2_fix: type fixed, parent right_index_link3, child right_index_tactile2, origin xyz=0 0 0 rpy=0 0 0, axis 0 0 0
- added joint right_index_tip_fix: type fixed, parent right_index_tactile2, child right_index_tip, origin xyz=0.027672 0.00055028 0 rpy=0 0 0, axis 0 0 0
- added joint right_middle_j0: type revolute, parent right_palm_base, child right_middle_link0, origin xyz=0.0071 0.011496 0.1218 rpy=0 -1.5708 0, axis 0 0 1, limit lower=-0.4363 upper=0.4363 effort=0 velocity=0
- added joint right_middle_j1: type revolute, parent right_middle_link0, child right_middle_link1, origin xyz=0.016 0 0 rpy=-1.5708 0 0, axis 0 0 1, limit lower=-0.349 upper=1.5707 effort=0 velocity=0
- added joint right_middle_j2: type revolute, parent right_middle_link1, child right_middle_link2, origin xyz=0.045 0 0 rpy=0 0 0, axis 0 0 1, limit lower=-0.0872 upper=1.7453 effort=0 velocity=0
- added joint right_middle_j3: type revolute, parent right_middle_link2, child right_middle_link3, origin xyz=0.025 0 0 rpy=0 0 0, axis 0 0 1, limit lower=-0.0872 upper=1.7453 effort=0 velocity=0, mimic joint=right_middle_j2 multiplier=1.0 offset=0
- added joint right_middle_pad_fix: type fixed, parent right_middle_tactile2, child right_middle_pad, origin xyz=0.017096144759137 0.00719554486026074 0 rpy=0 0 0, axis 0 0 0
- added joint right_middle_tactile0_fix: type fixed, parent right_middle_link1, child right_middle_tactile0, origin xyz=0 0 0 rpy=0 0 0, axis 0 0 0
- added joint right_middle_tactile1_fix: type fixed, parent right_middle_link2, child right_middle_tactile1, origin xyz=0 0 0 rpy=0 0 0, axis 0 0 0
- added joint right_middle_tactile2_fix: type fixed, parent right_middle_link3, child right_middle_tactile2, origin xyz=0 0 0 rpy=0 0 0, axis 0 0 0
- added joint right_middle_tip_fix: type fixed, parent right_middle_tactile2, child right_middle_tip, origin xyz=0.027672166719793 0.000550277924150981 0 rpy=0 0 0, axis 0 0 0
- added joint right_palm_base_fix: type fixed, parent right_palm_link, child right_palm_base, origin xyz=0 0 0 rpy=0 0 0, axis 0 0 0
- added joint right_palm_tactile_fix: type fixed, parent right_palm_link, child right_palm_tactile, origin xyz=0 0 0 rpy=0 0 0, axis 0 0 0
- added joint right_pinky_j0: type revolute, parent right_palm_base, child right_pinky_link0, origin xyz=0.0071 -0.034504 0.1158 rpy=0 -1.5708 0, axis 0 0 1, limit lower=-0.4363 upper=0.4363 effort=0 velocity=0
- added joint right_pinky_j1: type revolute, parent right_pinky_link0, child right_pinky_link1, origin xyz=0.016 0 0 rpy=-1.5708 0 0, axis 0 0 1, limit lower=-0.349 upper=1.5707 effort=0 velocity=0
- added joint right_pinky_j2: type revolute, parent right_pinky_link1, child right_pinky_link2, origin xyz=0.045 0 0 rpy=0 0 0, axis 0 0 1, limit lower=-0.0872 upper=1.7453 effort=0 velocity=0
- added joint right_pinky_j3: type revolute, parent right_pinky_link2, child right_pinky_link3, origin xyz=0.025 0 0 rpy=0 0 0, axis 0 0 1, limit lower=-0.0872 upper=1.7453 effort=0 velocity=0, mimic joint=right_pinky_j2 multiplier=1.0 offset=0
- added joint right_pinky_pad_fix: type fixed, parent right_pinky_tactile2, child right_pinky_pad, origin xyz=0.017096 0.0071955 0 rpy=0 0 0, axis 0 0 0
- added joint right_pinky_tactile0_fix: type fixed, parent right_pinky_link1, child right_pinky_tactile0, origin xyz=0 0 0 rpy=0 0 0, axis 0 0 0
- added joint right_pinky_tactile1_fix: type fixed, parent right_pinky_link2, child right_pinky_tactile1, origin xyz=0 0 0 rpy=0 0 0, axis 0 0 0
- added joint right_pinky_tactile2_fix: type fixed, parent right_pinky_link3, child right_pinky_tactile2, origin xyz=0 0 0 rpy=0 0 0, axis 0 0 0
- added joint right_pinky_tip_fix: type fixed, parent right_pinky_tactile2, child right_pinky_tip, origin xyz=0.027672 0.00055028 0 rpy=0 0 0, axis 0 0 0
- added joint right_ring_j0: type revolute, parent right_palm_base, child right_ring_link0, origin xyz=0.0071 -0.011503 0.1188 rpy=0 -1.5708 0, axis 0 0 1, limit lower=-0.4363 upper=0.4363 effort=0 velocity=0
- added joint right_ring_j1: type revolute, parent right_ring_link0, child right_ring_link1, origin xyz=0.016 0 0 rpy=-1.5708 0 0, axis 0 0 1, limit lower=-0.349 upper=1.5707 effort=0 velocity=0
- added joint right_ring_j2: type revolute, parent right_ring_link1, child right_ring_link2, origin xyz=0.045 0 0 rpy=0 0 0, axis 0 0 1, limit lower=-0.0872 upper=1.7453 effort=0 velocity=0
- added joint right_ring_j3: type revolute, parent right_ring_link2, child right_ring_link3, origin xyz=0.025 0 0 rpy=0 0 0, axis 0 0 1, limit lower=-0.0872 upper=1.7453 effort=0 velocity=0, mimic joint=right_ring_j2 multiplier=1.0 offset=0
- added joint right_ring_pad_fix: type fixed, parent right_ring_tactile2, child right_ring_pad, origin xyz=0.017096144759137 0.00719554486026074 0 rpy=0 0 0, axis 0 0 0
- added joint right_ring_tactile0_fix: type fixed, parent right_ring_link1, child right_ring_tactile0, origin xyz=0 0 0 rpy=0 0 0, axis 0 0 0
- added joint right_ring_tactile1_fix: type fixed, parent right_ring_link2, child right_ring_tactile1, origin xyz=0 0 0 rpy=0 0 0, axis 0 0 0
- added joint right_ring_tactile2_fix: type fixed, parent right_ring_link3, child right_ring_tactile2, origin xyz=0 0 0 rpy=0 0 0, axis 0 0 0
- added joint right_ring_tip_fix: type fixed, parent right_ring_tactile2, child right_ring_tip, origin xyz=0.027672166719793 0.000550277924150982 0 rpy=0 0 0, axis 0 0 0
- added joint right_thumb_j0: type revolute, parent right_palm_base, child right_thumb_link0, origin xyz=0.013 0.023 0.0493 rpy=3.1416 0 1.5708, axis 0 0 1, limit lower=0 upper=1.5707 effort=0 velocity=0
- added joint right_thumb_j1: type revolute, parent right_thumb_link0, child right_thumb_link1, origin xyz=0.0145 0 0 rpy=-1.5708 0 -1.5708, axis 0 0 1, limit lower=-0.1745 upper=1.0471 effort=0 velocity=0
- added joint right_thumb_j2: type revolute, parent right_thumb_link1, child right_thumb_link2, origin xyz=0 0 0.014 rpy=-1.5708 0 1.5708, axis 0 0 1, limit lower=0 upper=1.396 effort=0 velocity=0
- added joint right_thumb_j3: type revolute, parent right_thumb_link2, child right_thumb_link3, origin xyz=0 -0.055 0 rpy=0 0 -1.5708, axis 0 0 1, limit lower=-0.349 upper=1.396 effort=0 velocity=0
- added joint right_thumb_j4: type revolute, parent right_thumb_link3, child right_thumb_link4, origin xyz=0.03 0 0 rpy=0 0 0, axis 0 0 1, limit lower=-0.349 upper=1.396 effort=0 velocity=0, mimic joint=right_thumb_j3 multiplier=1.0 offset=0
- added joint right_thumb_pad_fix: type fixed, parent right_thumb_tactile2, child right_thumb_pad, origin xyz=0.018471 0.0088124 0 rpy=0 0 0, axis 0 0 0
- added joint right_thumb_tactile0_fix: type fixed, parent right_thumb_link2, child right_thumb_tactile0, origin xyz=0 0 0 rpy=0 0 0, axis 0 0 0
- added joint right_thumb_tactile1_fix: type fixed, parent right_thumb_link3, child right_thumb_tactile1, origin xyz=0 0 0 rpy=0 0 0, axis 0 0 0
- added joint right_thumb_tactile2_fix: type fixed, parent right_thumb_link4, child right_thumb_tactile2, origin xyz=0 0 0 rpy=0 0 0, axis 0 0 0
- added joint right_thumb_tip_fix: type fixed, parent right_thumb_tactile2, child right_thumb_tip, origin xyz=0.029863 -0.00039744 0 rpy=0 0 0, axis 0 0 0
